File: hardware/radio_board/radio.kicad_sch (KiCad schematic)
At the start: 29 parts, among them J2 RF, J3 Shield, U1 MAX2769B

Commit message: Add a clock distribution buffer to the radio board. See Issue #10
Parts:
- D2: LCSC C72043 -> C72038
- L1: value L -> LQG15HS33NG02D; LCSC (none) -> C3910755
