File: hardware/papilio_sodimm_interposer/connector.kicad_sch (KiCad schematic)
At the start: 1 part

Commit message: Got it going
Parts:
- added J1: Papilio Pro, Papilio_Pro:PAPILIO_PRO, symbol Papilio_pro:Papilio_Pro
Connections:
- new net: J1.3V3W1@1 (3.3V), J1.3V3W1@2 (3.3V), J1.3V3W1@3 (3.3V), J1.3V3W1@4 (3.3V), J1.3V3W2@1 (3.3V), J1.3V3W2@2 (3.3V)
- new net: J1.GNDW1@1 (GND), J1.GNDW1@2 (GND), J1.GNDW1@3 (GND), J1.GNDW1@4 (GND), J1.GNDW2@1 (GND), J1.GNDW2@2 (GND)
- new net: J1.VIW1@1 (5V), J1.VIW1@2 (5V), J1.VIW1@3 (5V), J1.VIW1@4 (5V), J1.VIW2@1 (5V), J1.VIW2@2 (5V)
